File: bbAutomationShield2.brd (EAGLE design)
At the start: 54.6 x 71.8 mm, 18 parts, among them U2 DHT22

Commit message: Changed board layout
http://letsmakerobots.com/files/userpics/u19048/B_3PinOut3.png

This pinout is INCORRECT
Parts:
- added E$19, E$20, E$21, E$9: (no value), adafruit:M0805
Routing:
- net S$10: track 83.8 -> 20.3 mm
- net S$63: track 56.5 -> 0.00 mm
- net S$61: track 52.8 -> 0.00 mm
- net S$59: track 51.6 -> 0.00 mm
- net S$62: track 50.0 -> 0.00 mm
- net S$60: track 48.7 -> 0.00 mm
- net N$28: track 0.00 -> 48.6 mm
- net N$34: track 0.00 -> 44.9 mm
- net S$41: track 44.6 -> 3.64 mm
- net S$48: track 40.8 -> 2.06 mm
- net N$30: track 0.00 -> 37.4 mm
- net S$40: track 53.5 -> 17.8 mm, vias 1 -> 0
- net S$58: track 46.8 -> 13.3 mm
- net S$2: track 42.6 -> 15.6 mm
- net S$14: track 0.00 -> 27.0 mm
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